File: hardware/due-laserscanning-powersupply/powersupply.sch (EAGLE design)
At the start: 14 parts, among them IC1 7805TV, X1 MKDSN1,5/3-5,08, X2 MKDSN1,5/2-5,08, X3 1751251, X4 BU-SMA-V, X5 BU-SMA-V, X6 BU-SMA-V, X7 MKDSN1,5/2-5,08

Commit message: update powersupply board
Parts:
- added C1, C2, C3, C4, C5, C6: (no value), rcl:C-EUC0805
- added X8: MKDSN1,5/2-5,08, con-phoenix-508:MKDSN1,5/2-5,08
Connections:
- net GND: now also C1.2, C2.2, C3.2, C4.2, C5.2, C6.2, X4.2, X5.2, X6.2, X8-1.KL
- net N$10: now also C3.1
- net N$6: now also X8-2.KL
- net N$7: now also C4.1, C5.1, C6.1
- net N$8: now also C1.1
- net N$9: now also C2.1
Changed lines of the file:
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@@
 <part name="P+4" library="supply1" deviceset="VCC" device=""/>
 <part name="GND9" library="supply1" deviceset="GND" device=""/>
+<part name="X8" library="con-phoenix-508" deviceset="MKDSN1,5/2-5,08" device=""/>
+<part name="GND10" library="supply1" deviceset="GND" device=""/>
+<part name="GND11" library="supply1" deviceset="GND" device=""/>
+<part name="GND12" library="supply1" deviceset="GND" device=""/>
+<part name="GND13" library="supply1" deviceset="GND" device=""/>
+<part name="C1" library="rcl" deviceset="C-EU" device="C0805"/>
+<part name="C2" library="rcl" deviceset="C-EU" device="C0805"/>
+<part name="C3" library="rcl" deviceset="C-EU" device="C0805"/>
+<part name="C4" library="rcl" deviceset="C-EU" device="C0805"/>
+<part name="C5" library="rcl" deviceset="C-EU" device="C0805"/>
+<part name="C6" library="rcl" deviceset="C-EU" device="C0805"/>
+<part name="GND14" library="supply1" deviceset="GND" device=""/>
+<part name="GND15" library="supply1" deviceset="GND" device=""/>
+<part name="GND16" library="supply1" deviceset="GND" device=""/>
+<part name="GND17" library="supply1" deviceset="GND" device=""/>
+<part name="GND18" library="supply1" deviceset="GND" device=""/>
+<part name="GND19" library="supply1" deviceset="GND" device=""/>
 </parts>
 <sheets>
@@
 <instance part="P+4" gate="VCC" x="-12.7" y="53.34"/>
 <instance part="GND9" gate="1" x="-12.7" y="35.56"/>
+<instance part="X8" gate="-1" x="55.88" y="114.3"/>
+<instance part="X8" gate="-2" x="55.88" y="121.92"/>
+<instance part="GND10" gate="1" x="53.34" y="109.22"/>
+<instance part="GND11" gate="1" x="200.66" y="96.52" rot="R180"/>
+<instance part="GND12" gate="1" x="200.66" y="58.42" rot="R180"/>
+<instance part="GND13" gate="1" x="200.66" y="22.86" rot="R180"/>
+<instance part="C1" gate="G$1" x="172.72" y="86.36"/>
+<instance part="C2" gate="G$1" x="175.26" y="48.26"/>
+<instance part="C3" gate="G$1" x="175.26" y="12.7"/>
+<instance part="C4" gate="G$1" x="129.54" y="88.9"/>
+<instance part="C5" gate="G$1" x="137.16" y="50.8"/>
+<instance part="C6" gate="G$1" x="134.62" y="15.24"/>
+<instance part="GND14" gate="1" x="129.54" y="81.28"/>
+<instance part="GND15" gate="1" x="172.72" y="78.74"/>
+<instance part="GND16" gate="1" x="175.26" y="40.64"/>
+<instance part="GND17" gate="1" x="137.16" y="43.18"/>
+<instance part="GND18" gate="1" x="134.62" y="7.62"/>
+<instance part="GND19" gate="1" x="175.26" y="5.08"/>
 </instances>
 <busses>
@@
 <pinref part="GND9" gate="1" pin="GND"/>
 </segment>
+<segment>
+<pinref part="X8" gate="-1" pin="KL"/>
+<pinref part="GND10" gate="1" pin="GND"/>
+<wire x1="53.34" y1="111.76" x2="53.34" y2="114.3" width="0.1524" layer="91"/>
+</segment>
+<segment>
+<pinref part="X4" gate="G$1" pin="2"/>
+<pinref part="GND11" gate="1" pin="GND"/>
+<wire x1="200.66" y1="93.98" x2="200.66" y2="91.44" width="0.1524" layer="91"/>
+</segment>
+<segment>
+<pinref part="X5" gate="G$1" pin="2"/>
+<pinref part="GND12" gate="1" pin="GND"/>
+<wire x1="200.66" y1="55.88" x2="200.66" y2="53.34" width="0.1524" layer="91"/>
+</segment>
+<segment>
+<pinref part="X6" gate="G$1" pin="2"/>
+<pinref part="GND13" gate="1" pin="GND"/>
+<wire x1="200.66" y1="20.32" x2="200.66" y2="17.78" width="0.1524" layer="91"/>
+</segment>
+<segment>
+<pinref part="C4" gate="G$1" pin="2"/>
+<pinref part="GND14" gate="1" pin="GND"/>
+</segment>
+<segment>
+<pinref part="C1" gate="G$1" pin="2"/>
+<pinref part="GND15" gate="1" pin="GND"/>
+</segment>
+<segment>
+<pinref part="C2" gate="G$1" pin="2"/>
+<pinref part="GND16" gate="1" pin="GND"/>
+</segment>
+<segment>
+<pinref part="C5" gate="G$1" pin="2"/>
+<pinref part="GND17" gate="1" pin="GND"/>
+</segment>
+<segment>
+<pinref part="C6" gate="G$1" pin="2"/>
+<pinref part="GND18" gate="1" pin="GND"/>
+</segment>
+<segment>
+<pinref part="C3" gate="G$1" pin="2"/>
+<pinref part="GND19" gate="1" pin="GND"/>
+</segment>
 </net>
 <net name="VCC" class="0">
@@
 <pinref part="X3" gate="-3" pin="K"/>
 <wire x1="48.26" y1="88.9" x2="45.72" y2="88.9" width="0.1524" layer="91"/>
-<wire x1="86.36" y1="91.44" x2="45.72" y2="91.44" width="0.1524" layer="91"/>
-<wire x1="45.72" y1="91.44" x2="45.72" y2="88.9" width="0.1524" layer="91"/>
+<wire x1="86.36" y1="91.44" x2="48.26" y2="91.44" width="0.1524" layer="91"/>
+<wire x1="48.26" y1="91.44" x2="45.72" y2="88.9" width="0.1524" layer="91"/>
 <pinref part="IC1" gate="A1" pin="VI"/>
+<wire x1="45.72" y1="88.9" x2="45.72" y2="121.92" width="0.1524" layer="91"/>
+<pinref part="X8" gate="-2" pin="KL"/>
+<wire x1="45.72" y1="121.92" x2="53.34" y2="121.92" width="0.1524" layer="91"/>
 </segment>
 </net>
@@
 <segment>
 <pinref part="U$4" gate="G$1" pin="VIN"/>
-<wire x1="106.68" y1="91.44" x2="134.62" y2="91.44" width="0.1524" layer="91"/>
+<wire x1="106.68" y1="91.44" x2="129.54" y2="91.44" width="0.1524" layer="91"/>
+<wire x1="129.54" y1="91.44" x2="134.62" y2="91.44" width="0.1524" layer="91"/>
 <wire x1="134.62" y1="91.44" x2="139.7" y2="91.44" width="0.1524" layer="91"/>
 <wire x1="134.62" y1="91.44" x2="134.62" y2="53.34" width="0.1524" layer="91"/>
 <pinref part="U$5" gate="G$1" pin="VIN"/>
-<wire x1="134.62" y1="53.34" x2="139.7" y2="53.34" width="0.1524" layer="91"/>
+<wire x1="134.62" y1="53.34" x2="137.16" y2="53.34" width="0.1524" layer="91"/>
+<wire x1="137.16" y1="53.34" x2="139.7" y2="53.34" width="0.1524" layer="91"/>
 <wire x1="134.62" y1="53.34" x2="134.62" y2="17.78" width="0.1524" layer="91"/>
 <pinref part="U$6" gate="G$1" pin="VIN"/>
 <wire x1="134.62" y1="17.78" x2="139.7" y2="17.78" width="0.1524" layer="91"/>
 <pinref part="IC1" gate="A1" pin="VO"/>
+<pinref part="C4" gate="G$1" pin="1"/>
+<junction x="129.54" y="91.44"/>
+<pinref part="C5" gate="G$1" pin="1"/>
+<junction x="137.16" y="53.34"/>
+<pinref part="C6" gate="G$1" pin="1"/>
+<junction x="134.62" y="17.78"/>
 </segment>
 </net>
@@
 <pinref part="U$4" gate="G$1" pin="VOUT"/>
 <pinref part="X4" gate="G$1" pin="1"/>
-<wire x1="200.66" y1="88.9" x2="170.18" y2="88.9" width="0.1524" layer="91"/>
+<wire x1="200.66" y1="88.9" x2="172.72" y2="88.9" width="0.1524" layer="91"/>
+<pinref part="C1" gate="G$1" pin="1"/>
+<wire x1="172.72" y1="88.9" x2="170.18" y2="88.9" width="0.1524" layer="91"/>
+<junction x="172.72" y="88.9"/>
 </segment>
 </net>
@@
 <pinref part="U$5" gate="G$1" pin="VOUT"/>
 <pinref part="X5" gate="G$1" pin="1"/>
-<wire x1="200.66" y1="50.8" x2="170.18" y2="50.8" width="0.1524" layer="91"/>
+<wire x1="200.66" y1="50.8" x2="175.26" y2="50.8" width="0.1524" layer="91"/>
+<pinref part="C2" gate="G$1" pin="1"/>
+<wire x1="175.26" y1="50.8" x2="170.18" y2="50.8" width="0.1524" layer="91"/>
+<junction x="175.26" y="50.8"/>
 </segment>
 </net>
@@
 <pinref part="U$6" gate="G$1" pin="VOUT"/>
 <pinref part="X6" gate="G$1" pin="1"/>
-<wire x1="200.66" y1="15.24" x2="170.18" y2="15.24" width="0.1524" layer="91"/>
-</segment>
-</net>
+<wire x1="200.66" y1="15.24" x2="175.26" y2="15.24" width="0.1524" layer="91"/>
+<pinref part="C3" gate="G$1" pin="1"/>
+<wire x1="175.26" y1="15.24" x2="170.18" y2="15.24" width="0.1524" layer="91"/>
+<junction x="175.26" y="15.24"/>
+</segment>
+</net>

Commit message: first revision of powersupply board was a total failure due to small holes and mirrored components
Parts:
- added C7, C8: 10u, rcl:CPOL-EUB
- added JP1: (no value), pinhead:PINHD-1X3
- added PL1: (no value), con-harting-v:10V
- added X10, X11: BU-SMA-V, con-coax:BU-SMA-V
- added X9: NEB21R, con-lumberg:NEB21R
Connections:
- removed net N$1: U$2.+VOUT, X2-2.KL
- removed net N$10: C3.1, U$6.VOUT, X6.1
- removed net N$2: U$2.-VOUT, X2-1.KL
- removed net N$3: U$1.-VOUT, X1-3.KL
- removed net N$4: U$1.COMMON, X1-2.KL
- removed net N$5: U$1.+VOUT, X1-1.KL
- removed net N$6: IC1.VI, U$3.VOUT, X3-3.K, X8-2.KL
- removed net N$7: C4.1, C5.1, C6.1, IC1.VO, U$4.VIN, U$5.VIN, U$6.VIN
- removed net N$8: C1.1, U$4.VOUT, X4.1
- removed net N$9: C2.1, U$5.VOUT, X5.1
- new net +5V: C4.1, C5.1, C6.1, C8.+, IC1.VO, U$4.VIN, U$5.VIN, U$6.VIN, X3-1.K
- new net -12V: PL1.2, U$1.-VOUT, X1-3.KL
- new net 12V: PL1.6, U$1.+VOUT, X1-1.KL
- new net 12VCOM: PL1.4, U$1.COMMON, X1-2.KL
- new net 2V5: C3.1, PL1.5, U$6.VOUT, X6.1
- new net 3V: C2.1, PL1.3, U$5.VOUT, X5.1
- new net 3V3: C1.1, PL1.1, U$4.VOUT, X4.1
- new net 5VCOM: PL1.8, U$2.-VOUT, X2-1.KL
- new net 5VISO: PL1.10, U$2.+VOUT, X2-2.KL
- new net 9V: C7.+, IC1.VI, PL1.7, U$3.VOUT, X3-3.K, X8-2.KL
- new net N$11: JP1.1, X7-1.KL
- new net N$12: JP1.3, X9.1
- net GND: now also C7.-, C8.-, PL1.9, U$4./SHDN, U$5./SHDN, U$6./SHDN, X10.1, X10.2, X11.1, X11.2, X9.3
- net VCC: now also JP1.2; no longer X7-1.KL
Other:
- moved on the sheet: C4, IC1, X3-1, X4, X5, X6, X7-1, X7-2
